File: CRASH-launcher/docs/kicad/CRASH_4-channel.sch (KiCad schematic (older format))
At the start: 27 parts, among them IC1 ATMEGA328P-PU, P1 CONN_3X2, P2 TTL Serial / Prog, SW1 SELECT_1, SW2 SELECT_2, SW3 SELECT_3, SW4 SELECT_4, SW5 SW_ARM, SW6 SW_FIRE, U1 RFM12B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

Commit message: - finished header connections - added LDO and caps - added battery and sense resistors - moved things around for clarity - now almost passes DRC check... antenna and ICSP 3.3V are only complaints
Parts:
- removed R4: R, symbol R
- removed U1: RFM12B, symbol RFM12
- added BT1: BATTERY, symbol BATTERY
- added C2, C5, C8: 0.1uF, symbol C
- added C6, C7: 100uF, symbol CP1
- added D1: DIODE, symbol DIODE
- added F1: POLYSWITCH, symbol FUSE
- added IC2: RFM12B, symbol RFM12B
- added R6, R7, R8: 47, symbol R
- added U2: LP2950, symbol LP2950
- D2: renamed from D1; value LED -> link/act LED
- D3: renamed from D2; value LED -> continuity-chan1_LED
- D4: renamed from D3; value LED -> continuity-chan2_LED
- D5: renamed from D4; value LED -> continuity-chan3_LED
- D6: renamed from D5; value LED -> continuity-chan4_LED
- R4: renamed from R?1; value R -> 47
- R5: value R -> 47
- renumbered C2 to C3, C3 to C4, P2 to P1, P1 to P2
Connections:
- wire segments 108 -> 122
- no-connect marks 0 -> 7
Other:
- note added: "BAT SENSE\nVoltage Divider"
- note added: "Note: All inputs \nuse AVR onboard \n20k pullups"
- moved on the sheet: C1, C3, C4, D2, D3, D4, D5, D6, IC1, L1, P1, P2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
