File: CRASH-launcher/docs/kicad/CRASH_relay_single_channel.sch (KiCad schematic (older format))
At the start: 0 parts

Commit message: arg
Parts:
- added D?: DIODE, symbol DIODE
- added IGNITER: R, symbol R
- added L?: INDUCTOR, symbol INDUCTOR
- added Q? (x3): FET_N, symbol FET_N
- added R? (x2): 2.2k, symbol R
- added R?, R??: 470, symbol R
- added R??: 1k, symbol R
- added R??: 3.9k, symbol R
- added R??: IGNITER, PAD, symbol IGNITER
- added U?: TSC888, SOT23-5, symbol TSC888
- added U?: 4052, symbol 4052
Connections:
- net labels added: +12V, GND, VCC
- wire segments 0 -> 30

Commit message: 
Parts:
- removed R?: 2.2k, symbol R
- removed U?: 4052, symbol 4052
- added D?: DIODE, symbol DIODE
Changed lines of the file:
@@
-EESchema Schematic File Version 2  date Mon 20 Feb 2012 04:56:42 PM MST
+EESchema Schematic File Version 2  date Fri 23 Mar 2012 11:21:48 PM MDT
 LIBS:bryan_custom
 LIBS:power
@@
 Sheet 3 5
 Title ""
-Date "14 feb 2012"
+Date "24 mar 2012"
 Rev ""
 Comp ""
@@
 $EndDescr
 Wire Wire Line
+	7400 4750 4700 4750
+Wire Wire Line
 	5950 1400 5950 1800
-Wire Wire Line
-	4800 4750 4700 4750
 Wire Wire Line
 	5600 4250 5600 4350
@@
 Wire Wire Line
 	7500 4150 7500 4050
-Wire Wire Line
-	7400 4750 6200 4750
 Wire Wire Line
 	7050 5950 7050 5650
@@
 Wire Wire Line
 	4700 4250 4700 4750
+Wire Wire Line
+	5200 4350 5200 4250
+Connection ~ 5200 4250
+$Comp
+L DIODE D?
+U 1 1 4F6D547B
+P 5400 4350
+F 0 "D?" H 5400 4450 40  0000 C CNN
+F 1 "DIODE" H 5400 4250 40  0000 C CNN
+	1    5400 4350
+	-1   0    0    -1
+$EndComp
 $Comp
 L IGNITER R??
@@
 	1    5950 1200
 	0    1    1    0
-$EndComp
-$Comp
-L 4052 U?
-U 1 1 4F2C9D90
-P 5500 5350
-F 0 "U?" H 5600 5350 60  0000 C CNN
-F 1 "4052" H 5600 5150 60  0000 C CNN
-	1    5500 5350
-	-1   0    0    -1
 $EndComp
 $Comp
@@
 $EndComp
 $Comp
-L R R?
-U 1 1 4F2C9CC0
-P 7600 4750
-F 0 "R?" H 7640 4820 50  0000 C CNN
-F 1 "2.2k" H 7630 4680 50  0000 C CNN
-	1    7600 4750
-	-1   0    0    1
-$EndComp
-$Comp
