File: CRASH-launcher/docs/kicad/CRASH_4-channel_controller.sch (KiCad schematic (older format))
At the start: 39 parts, among them IC1 ATMEGA328P-PU, IC2 RFM12B, P1 TTL Serial / Prog, P2 CONN_3X2, SW1 SELECT_1, SW2 SELECT_2, SW3 SELECT_3, SW4 SELECT_4, SW5 SW_ARM, SW6 SW_FIRE, U2 LP2950, X1 8MHz

Commit message: Schematic update
Parts:
- added D3: TVS Diode, symbol ZENER
- gave numbers to parts that had none: 1
Connections:
- net +3.3V: now also C8.2; no longer C8.1
- net at C2.1, IC1.1 ((PCINT14/RESET)PC6): now also P2.5, R1.2
- net at IC1.11 ((PCINT21/OC0B/T1)PD5): now also SW2.1; no longer SW1.1
- net at IC1.12 ((PCINT22/OC0A/AIN0)PD6): now also SW3.1; no longer SW2.1
- net at IC1.13 ((PCINT23/AIN1)PD7): now also SW4.1; no longer SW3.1
- net at IC1.14 ((PCINT0/CLKO/ICP1)PB0): now also SW5.1; no longer SW4.1
- net at IC1.24 ((PCINT9/ADC1)PC1): now also SW6.2; no longer D2.1 (A)
- net at IC1.5 ((PCINT19/OC2B/INT1)PD3): now also D2.1 (A); no longer SW5.1
- net at IC1.6 ((PCINT20/XCK/T0)PD4): now also SW1.1; no longer SW6.2
- net at U2.2 (GND): now also C6.2, C7.2, C8.1
- net at D1.1 (A), F1.1, R3.1: now also D1.2 (K)
- net at BT1.1 (+), F1.2: no longer D1.2 (K)
- new net: BT1.2 (-), D1.1 (A)
Other:
- moved on the sheet: C6, C7, C8, U2

Commit message: arg
Parts:
- removed C2: 0.1uF, symbol C
- removed C3: 22pF, symbol C
- removed D1: 1N4004, symbol DIODE
- removed IC1: ATMEGA328P-PU, DIL28, symbol ATMEGA328P-P
- removed IC2: RFM12B, symbol RFM12B
- removed P2: CONN_3X2, symbol CONN_3X2
- added C6: 22pF, symbol C
- added C8: 0.1uF, symbol C
- added D2: 1N4004, symbol DIODE
- added IC1: RFM12B, symbol RFM12B
- added IC2: ATMEGA328P-PU, DIL28, symbol ATMEGA328P-P
- added P1: CONN_3X2, symbol CONN_3X2
- renumbered C5 to C1, C6 to C2, C7 to C3, C8 to C4, C1 to C5, C4 to C7, D2 to D4, D3 to D5, D4 to D6, D5 to D7, D6 to D8, P1 to P2, R3 to R1, R1 to R3, SW5 to SW1, SW6 to SW2, SW1 to SW3, SW2 to SW4, SW3 to SW5, SW4 to SW6, U2 to U1
Connections:
- net +3.3V: now also IC1.9 (VDD), IC2.20 (AVCC), P1.2
- net at R3.2: now also C8.1, IC2.1 ((PCINT14/RESET)PC6), P1.5
- net at C7.2, X1.1: now also IC2.10 ((PCINT7/XTAL2/TOSC2)PB7)
- net at SW4.1: now also IC2.11 ((PCINT21/OC0B/T1)PD5)
- net at SW5.1: now also IC2.12 ((PCINT22/OC0A/AIN0)PD6)
- net at SW6.1: now also IC2.13 ((PCINT23/AIN1)PD7)
- net at SW1.1: now also IC2.14 ((PCINT0/CLKO/ICP1)PB0)
- net at SP1.1: now also IC2.15 ((PCINT1/OC1A)PB1)
- net at P2.5: now also IC2.2 ((PCINT16/RXD)PD0)
- net at R1.2, R2.1: now also IC2.23 ((PCINT8/ADC0)PC0)
- net at SW2.2: now also IC2.24 ((PCINT9/ADC1)PC1)
- net at D5.1 (A): now also IC2.25 ((PCINT10/ADC2)PC2)
- net at D6.1 (A): now also IC2.26 ((PCINT11/ADC3)PC3)
- net at D7.1 (A): now also IC2.27 ((PCINT12/SDA/ADC4)PC4)
- net at D8.1 (A): now also IC2.28 ((PCINT14/SCL/ADC5)PC5)
- net at P2.4: now also IC2.3 ((PCINT17/TXD)PD1)
- net at D4.1 (A): now also IC2.5 ((PCINT19/OC2B/INT1)PD3)
- net at SW3.1: now also IC2.6 ((PCINT20/XCK/T0)PD4)
- net at X1.2: now also C6.2, IC2.9 ((PCINT6/XTAL1/TOSC1)PB6)
- net at C7.1: now also C6.1
- net at L1.2: now also IC1.8 (ANT)
- net at P2.6: now also C8.2
- net at C2.1, U1.1 (VIN): now also D3.2 (K), D2.2 (K)
- net at D1.2 (K), F1.1, R1.1: now also D2.1 (A)
- new net: IC1.14 (nSEL), IC2.16 ((PCINT2/OC1B/SS)PB2)
- new net: IC1.12 (SDI), IC2.17 ((PCINT3/OC2A/MOSI)PB3), P1.4
- new net: IC1.1 (SDO), IC2.18 ((PCINT4/MISO)PB4), P1.1
- new net: IC1.13 (SCK), IC2.19 ((PCINT5/SCK)PB5), P1.3
- new net: IC2.21 (AREF), IC2.7 (VCC)
- new net: IC2.22 (GND), IC2.8 (GND)
- new net: IC1.2 (nIRQ), IC2.4 ((PCINT18/INT0)PD2)
- new net: IC1.10 (GND), IC1.7 (GND)
- no-connect marks 7 -> 9
Other:
- moved on the sheet: D3
