File: CRASH-launcher/docs/kicad/CRASH_4-channel_rackUnit.sch (KiCad schematic (older format))
At the start: 39 parts, among them IC1 ATMEGA328P-PU, IC2 RFM12B, P1 TTL Serial / Prog, P2 CONN_3X2, U2 LP2950, X1 8MHz

Commit message: Schematic update
Parts:
- added D3: TVS Diode, symbol ZENER
- added F?: FUSE, symbol FUSE
- C6: value 100uF -> 2200uF
- D1: value 1N4004 -> 1N5402
- D2: renamed from D?; value 1N4004 -> 1N5821
- gave numbers to parts that had none: 6
- renumbered MASTER_ARM_COIL to CHAN1_COIL, CHAN4_COIL to CHAN2_COIL, CHAN2_COIL to CHAN4_COIL, CHAN1_COIL to MASTER_ARM_COIL
Connections:
- net +3.3V: now also C8.2; no longer C8.1
- net at IC1.11 ((PCINT21/OC0B/T1)PD5): now also U1.4 (I4); no longer U1.1 (I1)
- net at IC1.12 ((PCINT22/OC0A/AIN0)PD6): now also U1.3 (I3); no longer U1.2 (I2)
- net at IC1.13 ((PCINT23/AIN1)PD7): now also U1.2 (I2); no longer U1.3 (I3)
- net at IC1.14 ((PCINT0/CLKO/ICP1)PB0): now also U1.1 (I1)
- net at IC1.5 ((PCINT19/OC2B/INT1)PD3): now also D?.1 (A), D?.2 (K); no longer U1.7 (I7)
- net at D1.2 (K), U2.1 (VIN): now also U1.9 (COM), D3.1 (A); no longer C6.1
- net at RSHUNT.1, U3.4 (Vm): now also F?.1; no longer R3.1
- net at BT1.1 (+), SW?.2: no longer D2.2 (K)
- net at D1.1 (A): now also D2.2 (K), R3.1, F?.2
- net at C6.2, C7.2: now also C8.1; no longer C8.2
- net at U1.10 (O7): no longer CHAN1_COIL.1
- net at U1.12 (O5): now also CHAN1_COIL.1
- net at U1.5 (I5): now also IC1.6 ((PCINT20/XCK/T0)PD4)
Other:
- note added: "NOTE: Current sense amp and\nsupporting components optional"
- moved on the sheet: BT1, C6, C7, C8, CHAN1_COIL, D2

Commit message: arg
Parts:
- removed C1, C5, C8: 0.1uF, symbol C
- removed C4: 22pF, symbol C
- removed C6: 2200uF, symbol CP1
- removed C7: 100uF, symbol CP1
- removed D2: 1N5821, symbol DIODE
- removed L1: ANTENNA, symbol INDUCTOR
- removed P1: TTL Serial / Prog, symbol CONN_6
- removed R1: 10k, symbol R
- removed R3: 39k, symbol R
- removed SP1: SPEAKER, symbol SPEAKER
- added C10: 100uF, symbol CP1
- added C11, C12, C13: 0.1uF, symbol C
- added C15: 22pF, symbol C
- added C9: 2200uF, symbol CP1
- added D11: 1N5821, symbol DIODE
- added K? (x3): CONN_3, symbol CONN_3
- added L2: ANTENNA, symbol INDUCTOR
- added P4: TTL Serial / Prog, symbol CONN_6
- added R11: 10k, symbol R
- added R9: 39k, symbol R
- added SP2: SPEAKER, symbol SPEAKER
- added U?: MAX6030, SOT-3, symbol MAX60XX
- gave numbers to parts that had none: 5
- renumbered BT1 to BT2, C3 to C14, C2 to C16, C9 to C17, CHAN1_COIL to CHAN1_COIL1, CHAN1_sense to CHAN1_sense1, CHAN2_COIL to CHAN2_COIL1, CHAN2_sense to CHAN2_sense1, CHAN3_COIL to CHAN3_COIL1, CHAN3_sense to CHAN3_sense1, CHAN4_COIL to CHAN4_COIL1, CHAN4_sense to CHAN4_sense1, D1 to D10, D3 to D9, IC2 to IC1, IC1 to IC3, MASTER_ARM_COIL to MASTER_ARM_COIL1, P2 to P3, R2 to R10, RSHUNT to RSHUNT1, U1 to U4, X1 to X2
Connections:
- wire segments 129 -> 164
Other:
- note added: "NOTE: Enhanced Voltage reference is \noptional. If not used, connect AVR \nAREF and TSC888 VIN to the digital\nsupply (3.3 to 3.6V)"
- moved on the sheet: F2, SW7

Commit message: :wq
Parts:
- removed K?: CONN_3, symbol CONN_3
- added K?: CONN_3, symbol CONN_3
- added SW?: SW_POWER, symbol SPST
Connections:
- wire segments 164 -> 133
Other:
- note removed: "NOTE: Enhanced Voltage reference is \noptional. If not used, connect AVR \nAREF and TSC888 VIN to the digital\nsupply (3.3 to 3.6V)"
- moved on the sheet: R?, SW?
