File: CRASH-launcher/docs/kicad-bryan_4chan/analog.sch (KiCad schematic (older format))
At the start: 18 parts, among them P301 CONN_8, U301 MCP3208

Commit message: 
Parts:
- removed P301: CONN_8, symbol CONN_8
- removed R301, R302, R303, R304, R305, R306, R307, R308, R309, R310, R311, R312, R313, R314, R315, R316: R, symbol R
- added R10, R11, R12, R5, R6, R7, R8, R9: R, symbol R
- renumbered U301 to U4
Connections:
- net labels added: VCC, adc.1, adc.2, adc.3, adc.4, adc.5, adc.6, adc.7, adc.8
- net labels removed: VDD
- wire segments 60 -> 43
Other:
- note removed: "Connectors are\n at +12V if igniter\nhas continuity\n"

Commit message: first REAL shot at PCB
Parts:
- removed R10, R11, R12, R5, R6, R7, R8, R9: R, symbol R
- U4: footprint DIP-16 -> DIP-18
Connections:
- net labels added: VDD
- net labels removed: VCC
- wire segments 43 -> 35
Changed lines of the file:
@@
-EESchema Schematic File Version 2  date Sat 05 May 2012 12:12:20 AM MDT
+EESchema Schematic File Version 2  date Fri 08 Jun 2012 10:29:21 PM MDT
 LIBS:bryan_custom
 LIBS:rfm12
@@
 Sheet 4 6
 Title ""
-Date "13 apr 2012"
+Date "8 jun 2012"
 Rev ""
 Comp ""
@@
 Comment4 ""
 $EndDescr
-$Comp
-L VCC #PWR022
-U 1 1 4F87B9F3
-P 6350 2900
-F 0 "#PWR022" H 6350 3000 30  0001 C CNN
-F 1 "VCC" H 6350 3000 30  0000 C CNN
-	1    6350 2900
-	1    0    0    -1
-$EndComp
-$Comp
-L R R5
-U 1 1 4F8659D4
-P 3800 2800
-F 0 "R5" H 3840 2870 50  0000 C CNN
-F 1 "R" H 3830 2730 50  0000 C CNN
-	1    3800 2800
-	-1   0    0    -1
-$EndComp
-$Comp
-L R R6
-U 1 1 4F8659D3
-P 3800 3050
-F 0 "R6" H 3840 3120 50  0000 C CNN
-F 1 "R" H 3830 2980 50  0000 C CNN
-	1    3800 3050
-	-1   0    0    -1
-$EndComp
-$Comp
-L R R7
-U 1 1 4F8659D2
-P 3800 3300
-F 0 "R7" H 3840 3370 50  0000 C CNN
-F 1 "R" H 3830 3230 50  0000 C CNN
-	1    3800 3300
-	-1   0    0    -1
-$EndComp
-$Comp
-L R R8
-U 1 1 4F8659D1
-P 3800 3550
-F 0 "R8" H 3840 3620 50  0000 C CNN
-F 1 "R" H 3830 3480 50  0000 C CNN
-	1    3800 3550
-	-1   0    0    -1
-$EndComp
-$Comp
-L R R9
-U 1 1 4F8659D0
-P 3800 3800
-F 0 "R9" H 3840 3870 50  0000 C CNN
-F 1 "R" H 3830 3730 50  0000 C CNN
-	1    3800 3800
-	-1   0    0    -1
-$EndComp
-$Comp
-L R R10
-U 1 1 4F8659CF
-P 3800 4050
-F 0 "R10" H 3840 4120 50  0000 C CNN
-F 1 "R" H 3830 3980 50  0000 C CNN
-	1    3800 4050
-	-1   0    0    -1
-$EndComp
-$Comp
-L R R11
-U 1 1 4F8659CE
-P 3800 4300
-F 0 "R11" H 3840 4370 50  0000 C CNN
-F 1 "R" H 3830 4230 50  0000 C CNN
-	1    3800 4300
-	-1   0    0    -1
-$EndComp
-$Comp
-L R R12
-U 1 1 4F8659CD
-P 3800 4550
-F 0 "R12" H 3840 4620 50  0000 C CNN
-F 1 "R" H 3830 4480 50  0000 C CNN
-	1    3800 4550
-	-1   0    0    -1
-$EndComp
+Connection ~ 6050 3300
 Wire Wire Line
-	4000 4550 4600 4550
+	6200 4450 6200 4200
 Wire Wire Line
-	4600 4550 4600 4200
-Wire Wire Line
-	4600 4200 4700 4200
-Wire Wire Line
-	4000 4050 4300 4050
-Wire Wire Line
-	4300 4050 4300 3900
-Wire Wire Line
-	4300 3900 4700 3900
-Wire Wire Line
-	4000 3550 4150 3550
-Wire Wire Line
-	4150 3550 4150 3600
-Wire Wire Line
-	4150 3600 4700 3600
-Wire Wire Line
-	4000 3050 4450 3050
-Wire Wire Line
-	4450 3050 4450 3300
-Wire Wire Line
-	4450 3300 4700 3300
-Wire Wire Line
-	4700 3150 4600 3150
-Wire Wire Line
-	4600 3150 4600 2800
-Wire Wire Line
-	4600 2800 4000 2800
-Wire Wire Line
-	4700 3450 4300 3450
-Wire Wire Line
-	4300 3450 4300 3300
-Wire Wire Line
-	4300 3300 4000 3300
-Wire Wire Line
-	4700 3750 4150 3750
-Wire Wire Line
-	4150 3750 4150 3800
-Wire Wire Line
-	4150 3800 4000 3800
-Wire Wire Line
-	4700 4050 4450 4050
-Wire Wire Line
-	4450 4050 4450 4300
-Wire Wire Line
-	4450 4300 4000 4300
-Wire Wire Line
-	3600 4550 2800 4550
-Wire Wire Line
-	3600 4050 2800 4050
-Wire Wire Line
-	3600 3550 2800 3550
-Wire Wire Line
-	3600 3050 2800 3050
-Wire Wire Line
-	3600 2800 2800 2800
-Wire Wire Line
-	3600 3300 2800 3300
-Wire Wire Line
-	3600 3800 2800 3800
-Wire Wire Line
-	3600 4300 2800 4300
-Text GLabel 2800 3800 0    60   BiDi ~ 0
-adc.5
-Text GLabel 2800 4050 0    60   BiDi ~ 0
-adc.6
-Text GLabel 2800 4300 0    60   BiDi ~ 0
-adc.7
-Text GLabel 2800 4550 0    60   BiDi ~ 0
-adc.8
-Text GLabel 2800 3550 0    60   BiDi ~ 0
-adc.4
-Text GLabel 2800 3300 0    60   BiDi ~ 0
-adc.3
-Text GLabel 2800 3050 0    60   BiDi ~ 0
-adc.2
-Text GLabel 2800 2800 0    60   BiDi ~ 0
-adc.1
+	6200 4200 6050 4200
 Wire Wire Line
 	7000 3550 7000 3450
@@
 	7000 3450 6050 3450
 Wire Wire Line
-	6050 4050 6350 4050
+	6050 3900 6350 3900
+Wire Wire Line
+	6050 3600 6350 3600
+Wire Wire Line
+	6350 2900 6350 3150
+Wire Wire Line
+	6350 3150 6050 3150
+Wire Wire Line
+	6050 3300 6350 3300
 Wire Wire Line
 	6050 3750 6350 3750
 Wire Wire Line
-	6050 3300 6350 3300
+	4000 4300 4450 4300
 Wire Wire Line
-	6050 3150 6350 3150
+	4450 4300 4450 4050
 Wire Wire Line
-	6350 3150 6350 2900
+	4450 4050 4700 4050
 Wire Wire Line
-	6050 3600 6350 3600
+	4000 3800 4150 3800
 Wire Wire Line
-	6050 3900 6350 3900
+	4150 3800 4150 3750
 Wire Wire Line
-	6050 4200 6200 4200
+	4150 3750 4700 3750
 Wire Wire Line
-	6200 4200 6200 4450
+	4000 3300 4300 3300
+Wire Wire Line
+	4300 3300 4300 3450
+Wire Wire Line
+	4300 3450 4700 3450
+Wire Wire Line
+	4000 2800 4600 2800
+Wire Wire Line
+	4600 2800 4600 3150
+Wire Wire Line
+	4600 3150 4700 3150
+Wire Wire Line
+	4700 3300 4450 3300
+Wire Wire Line
+	4450 3300 4450 3050
+Wire Wire Line
+	4450 3050 4000 3050
+Wire Wire Line
+	4700 3600 4150 3600
+Wire Wire Line
+	4150 3600 4150 3550
+Wire Wire Line
+	4150 3550 4000 3550
+Wire Wire Line
+	4700 3900 4300 3900
+Wire Wire Line
+	4300 3900 4300 4050
+Wire Wire Line
+	4300 4050 4000 4050
+Wire Wire Line
+	4700 4200 4600 4200
+Wire Wire Line
+	4600 4200 4600 4550
+Wire Wire Line
+	4600 4550 4000 4550
+Wire Wire Line
+	6050 4050 6350 4050
 $Comp
-L GND #U023
-U 1 1 4F25EE8A
+L VDD #PWR035
+U 1 1 4FCD3FFB
+P 6350 2900
+F 0 "#PWR035" H 6350 3000 30  0001 C CNN
+F 1 "VDD" H 6350 3010 30  0000 C CNN
+	1    6350 2900
+	1    0    0    -1
+$EndComp
+$Comp
+L GND #PWR036
+U 1 1 4FCC1CD3
 P 6200 4450
-F 0 "#U023" H 6250 4500 60  0001 C CNN
-F 1 "GND" H 6200 4215 60  0000 C CNN
+F 0 "#PWR036" H 6200 4450 30  0001 C CNN
+F 1 "GND" H 6200 4380 30  0001 C CNN
 	1    6200 4450
 	1    0    0    -1
 $EndComp
+Text GLabel 4000 3800 0    60   BiDi ~ 0
+adc.5
+Text GLabel 4000 4050 0    60   BiDi ~ 0
+adc.6
+Text GLabel 4000 4300 0    60   BiDi ~ 0
+adc.7
+Text GLabel 4000 4550 0    60   BiDi ~ 0
+adc.8
+Text GLabel 4000 3550 0    60   BiDi ~ 0
+adc.4
+Text GLabel 4000 3300 0    60   BiDi ~ 0
+adc.3
+Text GLabel 4000 3050 0    60   BiDi ~ 0
+adc.2
+Text GLabel 4000 2800 0    60   BiDi ~ 0
+adc.1
 $Comp
-L GND #U024
+L GND #U037
 U 1 1 4F25EE87
 P 7000 3550
-F 0 "#U024" H 7050 3600 60  0001 C CNN
+F 0 "#U037" H 7050 3600 60  0001 C CNN
 F 1 "GND" H 7000 3315 60  0000 C CNN
 	1    7000 3550
@@
 F 0 "U4" H 5750 4450 60  0000 C CNN
 F 1 "MCP3208" H 5350 3000 60  0000 C CNN
-F 2 "DIP-16" H 5100 4450 60  0000 C CNN
+F 2 "DIP-18" H 5100 4450 60  0000 C CNN
 	1    5350 3700
 	1    0    0    -1

Commit message: second try at PCB layout.  this one might actually work!
Parts:
- added K10: CONN_3, symbol CONN_3
- added P11: CONN_5, symbol CONN_5
- added RR1: RR8, symbol RR8
Connections:
- net VDD: now also RR1.9
- net adc.1: now also K10.3 (P3), RR1.1 (COM)
- net adc.2: now also K10.2 (PM), RR1.2
- net adc.3: now also K10.1 (P1), RR1.3
- net adc.4: now also P11.5, RR1.4
- net adc.5: now also P11.4, RR1.5
- net adc.6: now also P11.3, RR1.6
- net adc.7: now also P11.2, RR1.7
- net adc.8: now also P11.1, RR1.8
Changed lines of the file:
@@
-EESchema Schematic File Version 2  date Fri 08 Jun 2012 10:29:21 PM MDT
+EESchema Schematic File Version 2  date Sun 10 Jun 2012 01:48:40 AM MDT
 LIBS:bryan_custom
 LIBS:rfm12
@@
 Sheet 4 6
 Title ""
-Date "8 jun 2012"
+Date "10 jun 2012"
 Rev ""
 Comp ""
@@
 Comment4 ""
 $EndDescr
+$Comp
+L CONN_3 K10
+U 1 1 4FD3DBC5
+P 3900 5050
+F 0 "K10" V 3850 5050 50  0000 C CNN
+F 1 "CONN_3" V 3950 5050 40  0000 C CNN
+	1    3900 5050
+	0    1    1    0
+$EndComp
+$Comp
+L CONN_5 P11
+U 1 1 4FD3DBBF
+P 4300 5100
+F 0 "P11" V 4250 5100 50  0000 C CNN
+F 1 "CONN_5" V 4350 5100 50  0000 C CNN
+	1    4300 5100
+	0    1    1    0
+$EndComp
+Connection ~ 3800 3150
+Wire Wire Line
+	3800 4700 3800 2700
+Wire Wire Line
+	4000 4700 4000 2700
+Wire Wire Line
+	4200 4700 4200 2700
+Wire Wire Line
+	4400 4700 4400 2700
+Connection ~ 3800 2800
+Connection ~ 4000 3450
+Connection ~ 4200 3750
+Connection ~ 4400 4050
+Wire Wire Line
+	4600 2700 6100 2700
+Wire Wire Line
+	4700 4050 3600 4050
+Wire Wire Line
+	4700 3750 3350 3750
+Wire Wire Line
+	4700 3450 3500 3450
+Wire Wire Line
+	3800 3150 4700 3150
 Connection ~ 6050 3300
 Wire Wire Line
@@
 	6050 3750 6350 3750
 Wire Wire Line
-	4000 4300 4450 4300
-Wire Wire Line
-	4450 4300 4450 4050
-Wire Wire Line
-	4450 4050 4700 4050
-Wire Wire Line
-	4000 3800 4150 3800
-Wire Wire Line
-	4150 3800 4150 3750
-Wire Wire Line
-	4150 3750 4700 3750
-Wire Wire Line
-	4000 3300 4300 3300
-Wire Wire Line
-	4300 3300 4300 3450
-Wire Wire Line
-	4300 3450 4700 3450
-Wire Wire Line
-	4000 2800 4600 2800
-Wire Wire Line
-	4600 2800 4600 3150
-Wire Wire Line
-	4600 3150 4700 3150
-Wire Wire Line
-	4700 3300 4450 3300
-Wire Wire Line
-	4450 3300 4450 3050
-Wire Wire Line
-	4450 3050 4000 3050
-Wire Wire Line
-	4700 3600 4150 3600
-Wire Wire Line
-	4150 3600 4150 3550
-Wire Wire Line
-	4150 3550 4000 3550
-Wire Wire Line
-	4700 3900 4300 3900
-Wire Wire Line
-	4300 3900 4300 4050
-Wire Wire Line
-	4300 4050 4000 4050
-Wire Wire Line
-	4700 4200 4600 4200
-Wire Wire Line
-	4600 4200 4600 4550
-Wire Wire Line
-	4600 4550 4000 4550
+	3200 4300 3600 4300
+Wire Wire Line
+	3600 4300 3600 4050
+Wire Wire Line
+	3200 3800 3350 3800
+Wire Wire Line
+	3350 3800 3350 3750
+Wire Wire Line
+	3200 3300 3500 3300
+Wire Wire Line
+	3500 3300 3500 3450
+Wire Wire Line
+	3200 2800 3800 2800
+Wire Wire Line
+	3650 3050 3650 3300
+Wire Wire Line
+	3650 3050 3200 3050
+Wire Wire Line
+	3350 3550 3350 3600
+Wire Wire Line
+	3350 3550 3200 3550
+Wire Wire Line
+	3500 4050 3500 3900
+Wire Wire Line
+	3500 4050 3200 4050
+Wire Wire Line
+	3700 4550 3700 4200
+Wire Wire Line
+	3700 4550 3200 4550
 Wire Wire Line
 	6050 4050 6350 4050
+Wire Wire Line
+	6350 2950 6100 2950
+Connection ~ 6350 2950
+Wire Wire Line
+	6100 2950 6100 2700
+Wire Wire Line
+	3650 3300 4700 3300
+Wire Wire Line
+	3350 3600 4700 3600
+Wire Wire Line
+	3500 3900 4700 3900
+Wire Wire Line
+	3700 4200 4700 4200
+Connection ~ 4500 4200
+Connection ~ 4300 3900
+Connection ~ 4100 3600
+Connection ~ 3900 3300
+Wire Wire Line
+	4500 4700 4500 2700
+Wire Wire Line
+	4300 4700 4300 2700
+Wire Wire Line
+	4100 4700 4100 2700
+Wire Wire Line
+	3900 4700 3900 2700
+$Comp
+L RR8 RR1
+U 1 1 4FD3D4A2
+P 4250 2350
+F 0 "RR1" H 4300 2900 70  0000 C CNN
+F 1 "RR8" V 4280 2350 70  0000 C CNN
+	1    4250 2350
+	0    -1   -1   0
+$EndComp
 $Comp
 L VDD #PWR035
@@
 	1    0    0    -1
 $EndComp
-Text GLabel 4000 3800 0    60   BiDi ~ 0
+Text GLabel 3200 3800 0    60   BiDi ~ 0
 adc.5
-Text GLabel 4000 4050 0    60   BiDi ~ 0
+Text GLabel 3200 4050 0    60   BiDi ~ 0
 adc.6
-Text GLabel 4000 4300 0    60   BiDi ~ 0
+Text GLabel 3200 4300 0    60   BiDi ~ 0
 adc.7
-Text GLabel 4000 4550 0    60   BiDi ~ 0
+Text GLabel 3200 4550 0    60   BiDi ~ 0
 adc.8
-Text GLabel 4000 3550 0    60   BiDi ~ 0
+Text GLabel 3200 3550 0    60   BiDi ~ 0
 adc.4
-Text GLabel 4000 3300 0    60   BiDi ~ 0
+Text GLabel 3200 3300 0    60   BiDi ~ 0
 adc.3
-Text GLabel 4000 3050 0    60   BiDi ~ 0
+Text GLabel 3200 3050 0    60   BiDi ~ 0
 adc.2
-Text GLabel 4000 2800 0    60   BiDi ~ 0
+Text GLabel 3200 2800 0    60   BiDi ~ 0
 adc.1
 $Comp
