File: CRASH-launcher/docs/kicad-bryan_4chan/analog.sch (KiCad schematic (older format))
At the start: 4 parts, among them K10 CONN_3, P11 CONN_5, U4 MCP3208

Commit message: rounded corners, plopped in a few missing caps on gpios and adc
Parts:
- added C18, C19: 0.1uF, symbol C
Connections:
- net GND: now also C18.1, C19.2
- net VDD: now also C18.2
- net VREF: now also C19.1
Changed lines of the file:
@@
-EESchema Schematic File Version 2  date Wed 13 Jun 2012 10:43:09 PM MDT
+EESchema Schematic File Version 2  date Fri 06 Jul 2012 11:04:22 PM MDT
 LIBS:bryan_custom
 LIBS:rfm12
@@
 Sheet 4 6
 Title ""
-Date "11 jun 2012"
+Date "7 jul 2012"
 Rev ""
 Comp ""
@@
 Comment4 ""
 $EndDescr
+Wire Wire Line
+	6100 2300 6100 2050
+Wire Wire Line
+	7000 3950 7000 3450
+Connection ~ 6100 2700
+Connection ~ 3800 3150
+Wire Wire Line
+	3800 4700 3800 2700
+Wire Wire Line
+	4000 4700 4000 2700
+Wire Wire Line
+	4200 4700 4200 2700
+Wire Wire Line
+	4400 4700 4400 2700
+Connection ~ 3800 2800
+Connection ~ 4000 3450
+Connection ~ 4200 3750
+Connection ~ 4400 4050
+Wire Wire Line
+	4600 2700 6100 2700
+Wire Wire Line
+	4700 4050 3600 4050
+Wire Wire Line
+	4700 3750 3350 3750
+Wire Wire Line
+	4700 3450 3500 3450
+Wire Wire Line
+	3800 3150 4700 3150
+Connection ~ 6050 3300
+Wire Wire Line
+	6200 4450 6200 4200
+Wire Wire Line
+	6200 4200 6050 4200
+Wire Wire Line
+	7000 3450 6050 3450
+Wire Wire Line
+	6050 3900 6350 3900
+Wire Wire Line
+	6050 3600 6350 3600
+Wire Wire Line
+	6350 2900 6350 3150
+Wire Wire Line
+	6350 3150 6050 3150
+Wire Wire Line
+	6050 3750 6350 3750
+Wire Wire Line
+	3200 4300 3600 4300
+Wire Wire Line
+	3600 4300 3600 4050
+Wire Wire Line
+	3200 3800 3350 3800
+Wire Wire Line
+	3350 3800 3350 3750
+Wire Wire Line
+	3200 3300 3500 3300
+Wire Wire Line
+	3500 3300 3500 3450
+Wire Wire Line
+	3200 2800 3800 2800
+Wire Wire Line
+	3650 3050 3650 3300
+Wire Wire Line
+	3650 3050 3200 3050
+Wire Wire Line
+	3350 3550 3350 3600
+Wire Wire Line
+	3350 3550 3200 3550
+Wire Wire Line
+	3500 4050 3500 3900
+Wire Wire Line
+	3500 4050 3200 4050
+Wire Wire Line
+	3700 4550 3700 4200
+Wire Wire Line
+	3700 4550 3200 4550
+Wire Wire Line
+	6050 4050 6350 4050
+Wire Wire Line
+	6350 2950 6100 2950
+Connection ~ 6350 2950
+Wire Wire Line
+	6100 2950 6100 2700
+Wire Wire Line
+	3650 3300 4700 3300
+Wire Wire Line
+	3350 3600 4700 3600
+Wire Wire Line
+	3500 3900 4700 3900
+Wire Wire Line
+	3700 4200 4700 4200
+Connection ~ 4500 4200
+Connection ~ 4300 3900
+Connection ~ 4100 3600
+Connection ~ 3900 3300
+Wire Wire Line
+	4500 4700 4500 2700
+Wire Wire Line
+	4300 4700 4300 2700
+Wire Wire Line
+	4100 4700 4100 2700
+Wire Wire Line
+	3900 4700 3900 2700
+Wire Wire Line
+	7500 3300 6050 3300
+Wire Wire Line
+	7350 3700 7000 3700
+Connection ~ 7000 3700
+Connection ~ 7350 3300
+$Comp
+L GND #U034
+U 1 1 4FF7BDAE
+P 6100 2050
+F 0 "#U034" H 6150 2100 60  0001 C CNN
+F 1 "GND" H 6100 1815 60  0000 C CNN
+	1    6100 2050
+	-1   0    0    1
+$EndComp
+$Comp
+L C C19
+U 1 1 4FF7BD94
+P 7350 3500
+F 0 "C19" H 7400 3600 50  0000 L CNN
+F 1 "0.1uF" H 7400 3400 50  0000 L CNN
+	1    7350 3500
+	1    0    0    -1
+$EndComp
+$Comp
+L C C18
+U 1 1 4FF7BD7A
+P 6100 2500
+F 0 "C18" H 6150 2600 50  0000 L CNN
+F 1 "0.1uF" H 6150 2400 50  0000 L CNN
+	1    6100 2500
+	1    0    0    -1
+$EndComp
 $Comp
 L CONN_3 K10
@@
 	0    1    1    0
 $EndComp
-Connection ~ 3800 3150
-Wire Wire Line
-	3800 4700 3800 2700
-Wire Wire Line
-	4000 4700 4000 2700
-Wire Wire Line
-	4200 4700 4200 2700
-Wire Wire Line
-	4400 4700 4400 2700
-Connection ~ 3800 2800
-Connection ~ 4000 3450
-Connection ~ 4200 3750
-Connection ~ 4400 4050
-Wire Wire Line
-	4600 2700 6100 2700
-Wire Wire Line
-	4700 4050 3600 4050
-Wire Wire Line
-	4700 3750 3350 3750
-Wire Wire Line
-	4700 3450 3500 3450
-Wire Wire Line
-	3800 3150 4700 3150
-Connection ~ 6050 3300
-Wire Wire Line
-	6200 4450 6200 4200
-Wire Wire Line
-	6200 4200 6050 4200
-Wire Wire Line
-	7000 3550 7000 3450
-Wire Wire Line
-	7000 3450 6050 3450
-Wire Wire Line
-	6050 3900 6350 3900
-Wire Wire Line
-	6050 3600 6350 3600
-Wire Wire Line
-	6350 2900 6350 3150
-Wire Wire Line
-	6350 3150 6050 3150
-Wire Wire Line
-	6050 3300 6350 3300
-Wire Wire Line
-	6050 3750 6350 3750
-Wire Wire Line
-	3200 4300 3600 4300
-Wire Wire Line
-	3600 4300 3600 4050
-Wire Wire Line
-	3200 3800 3350 3800
-Wire Wire Line
-	3350 3800 3350 3750
-Wire Wire Line
-	3200 3300 3500 3300
-Wire Wire Line
-	3500 3300 3500 3450
-Wire Wire Line
-	3200 2800 3800 2800
-Wire Wire Line
-	3650 3050 3650 3300
-Wire Wire Line
-	3650 3050 3200 3050
-Wire Wire Line
-	3350 3550 3350 3600
-Wire Wire Line
-	3350 3550 3200 3550
-Wire Wire Line
-	3500 4050 3500 3900
-Wire Wire Line
-	3500 4050 3200 4050
-Wire Wire Line
-	3700 4550 3700 4200
-Wire Wire Line
-	3700 4550 3200 4550
-Wire Wire Line
-	6050 4050 6350 4050
-Wire Wire Line
-	6350 2950 6100 2950
-Connection ~ 6350 2950
-Wire Wire Line
-	6100 2950 6100 2700
-Wire Wire Line
-	3650 3300 4700 3300
-Wire Wire Line
-	3350 3600 4700 3600
-Wire Wire Line
-	3500 3900 4700 3900
-Wire Wire Line
-	3700 4200 4700 4200
-Connection ~ 4500 4200
-Connection ~ 4300 3900
-Connection ~ 4100 3600
-Connection ~ 3900 3300
-Wire Wire Line
-	4500 4700 4500 2700
-Wire Wire Line
-	4300 4700 4300 2700
-Wire Wire Line
-	4100 4700 4100 2700
-Wire Wire Line
-	3900 4700 3900 2700
 $Comp
 L RR8 RR1
@@
 $EndComp
 $Comp
-L VDD #PWR038
+L VDD #PWR035
 U 1 1 4FCD3FFB
 P 6350 2900
-F 0 "#PWR038" H 6350 3000 30  0001 C CNN
+F 0 "#PWR035" H 6350 3000 30  0001 C CNN
 F 1 "VDD" H 6350 3010 30  0000 C CNN
 	1    6350 2900
@@
 $EndComp
 $Comp
-L GND #PWR039
+L GND #PWR036
 U 1 1 4FCC1CD3
 P 6200 4450
-F 0 "#PWR039" H 6200 4450 30  0001 C CNN
+F 0 "#PWR036" H 6200 4450 30  0001 C CNN
 F 1 "GND" H 6200 4380 30  0001 C CNN
 	1    6200 4450
@@
 adc.1
 $Comp
-L GND #U040
+L GND #U037
 U 1 1 4F25EE87
-P 7000 3550
-F 0 "#U040" H 7050 3600 60  0001 C CNN
-F 1 "GND" H 7000 3315 60  0000 C CNN
-	1    7000 3550
+P 7000 3950
+F 0 "#U037" H 7050 4000 60  0001 C CNN
+F 1 "GND" H 7000 3715 60  0000 C CNN
+	1    7000 3950
 	1    0    0    -1
 $EndComp
@@
 Text HLabel 6350 3750 2    60   Input ~ 12
 MISO
-Text HLabel 6350 3300 2    60   Input ~ 12
+Text HLabel 7500 3300 2    60   Input ~ 12
 VREF
 Text HLabel 6350 3600 2    60   Input ~ 12
