File: CRASH-launcher/docs/kicad-bryan_4chan/gpios.sch (KiCad schematic (older format))
At the start: 32 parts, among them U401 MCP23S17, U402 MCP23S17

Commit message: 
Parts:
- removed LED401, LED402, LED403, LED404: LED_RCGB, symbol LED_RCGB
- removed R401, R402, R403, R404, R405, R406, R407, R408, R409, R410, R411, R412, R413, R414, R415, R416: R, symbol R
- added R13, R14, R15, R16, R17, R18, R19, R20, R21, R22, R23, R24, R25, R26, R27, R28, R30, R32, R34, R36, R38, R40, R42, R44: R, symbol R
- renumbered R417 to R29, R418 to R31, R419 to R33, R420 to R35, R421 to R37, R422 to R39, R423 to R41, R424 to R43, R425 to R45, R426 to R46, U401 to U5, U402 to U6
Connections:
- net labels added: VCC, gpa.1, gpa.10, gpa.11, gpa.12, gpa.13, gpa.14, gpa.15, gpa.16, gpa.2, gpa.3, gpa.4, gpa.5, gpa.6, gpa.7, gpa.8, gpa.9, gpb.1, gpb.10, gpb.11, gpb.12, gpb.13, gpb.14, gpb.15, gpb.16, gpb.2, gpb.3, gpb.4, gpb.5, gpb.6, gpb.7, gpb.8, gpb.9
- net labels removed: +3.3V
- wire segments 138 -> 144

Commit message: first REAL shot at PCB
Parts:
- removed R13, R14, R15, R16, R17, R18, R19, R20, R21, R22, R23, R24, R25, R26, R27, R28, R30, R31, R32, R33, R34, R35, R36, R37, R38, R39, R40, R41, R42, R43, R44, R45: R, symbol R
- added P12, P13, P14: CONN_2X8, symbol CONN_2X8
- added U5, U6, U8, U9: ULN2803A, DIP-18, symbol ULN2803A
- renumbered R29 to R5, R46 to R6, U6 to U10, U5 to U7
Connections:
- net labels added: +12V, VDD
- net labels removed: VCC
- wire segments 144 -> 147
- no-connect marks 0 -> 6
Other:
- moved on the sheet: R5, R6, U10, U7

Commit message: second try at PCB layout.  this one might actually work!
Parts:
- removed P12: CONN_2X8, symbol CONN_2X8
- added K4, K5, K6, K7: CONN_3, symbol CONN_3
- added P25: CONN_2X8, symbol CONN_2X8
- added R10, R11: 10k, symbol R
Connections:
- net +12V: now also K4.1 (P1), K5.1 (P1), K6.1 (P1), K7.1 (P1); no longer U5.10 (COM), U6.10 (COM), U8.10 (COM), U9.10 (COM)
- net GND: now also R10.2, R11.2
- net VDD: now also K4.3 (P3), K5.3 (P3), K6.3 (P3), K7.3 (P3)
- net gpa.1: now also U5.11 (OUT8); no longer U5.18 (OUT1)
- net gpa.10: now also P25.10
- net gpa.11: now also P25.11
- net gpa.12: now also P25.12
- net gpa.13: now also P25.13
- net gpa.14: now also P25.14
- net gpa.15: now also P25.15
- net gpa.16: now also P25.16
- net gpa.2: now also U5.12 (OUT7); no longer U5.17 (OUT2)
- net gpa.3: now also U5.13 (OUT6); no longer U5.16 (OUT3)
- net gpa.4: now also U5.14 (OUT5); no longer U5.15 (OUT4)
- net gpa.5: now also U5.15 (OUT4); no longer U5.14 (OUT5)
- net gpa.6: now also U5.16 (OUT3); no longer U5.13 (OUT6)
- net gpa.7: now also U5.17 (OUT2); no longer U5.12 (OUT7)
- net gpa.8: now also U5.18 (OUT1); no longer U5.11 (OUT8)
- net gpa.9: now also P25.9
- net GPIO_RESET: now reaches U7.18 (RESET)
- net GPIO_RESET: now also U10.18 (RESET), R10.1, R11.1
- net at U10.21 (GPA0): now also U9.1 (IN1); no longer U9.8 (IN8)
- net at U10.22 (GPA1): now also U9.2 (IN2); no longer U9.7 (IN7)
- net at U10.23 (GPA2): now also U9.3 (IN3); no longer U9.6 (IN6)
- net at U10.24 (GPA3): now also U9.4 (IN4); no longer U9.5 (IN5)
- net at U10.25 (GPA4): now also U9.5 (IN5); no longer U9.4 (IN4)
- net at U10.26 (GPA5): now also U9.6 (IN6); no longer U9.3 (IN3)
- net at U10.27 (GPA6): now also U9.7 (IN7); no longer U9.2 (IN2)
- net at U10.28 (GPA7): now also U9.8 (IN8); no longer U9.1 (IN1)
- net at U6.11 (OUT8): now also P25.8
- net at U6.12 (OUT7): now also P25.7
- net at U6.13 (OUT6): now also P25.6
- net at U6.14 (OUT5): now also P25.5
- net at U6.15 (OUT4): now also P25.4
- net at U6.16 (OUT3): now also P25.3
- net at U6.17 (OUT2): now also P25.2
- net at U6.18 (OUT1): now also P25.1
- new net: K4.2 (PM), U5.10 (COM)
- new net: K7.2 (PM), U9.10 (COM)
- new net: K6.2 (PM), U8.10 (COM)
- new net: K5.2 (PM), U6.10 (COM)
- no-connect marks 6 -> 4
Other:
- moved on the sheet: U9
