File: CRASH-launcher/docs/kicad-bryan_4chan/gpios.sch (KiCad schematic (older format))
At the start: 17 parts, among them K4 CONN_3, K5 CONN_3, K6 CONN_3, K7 CONN_3, P13 CONN_2X8, P14 CONN_2X8, P25 CONN_2X8, U10 MCP23S17, U5 ULN2803A, U6 ULN2803A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

Commit message: rounded corners, plopped in a few missing caps on gpios and adc
Parts:
- added C16, C17: 0.1uF, symbol C
Connections:
- net GND: now also C16.2, C17.2
- net VDD: now also C16.1, C17.1
