File: CRASH-launcher/docs/kicad-bryan_4chan/power.sch (KiCad schematic (older format))
At the start: 16 parts, among them SW201 SW_POWER, U201 LP2950, U202 TSC888, U203 MAX6030

Commit message: 
Parts:
- removed D203: 1N5821, symbol DIODE
- removed U203: MAX6030, SOT-3, symbol MAX60XX
- added C4, C6: 3300uF, symbol CP1
- added C5, C8: 0.1uF, symbol C
- added C7: 470uF, symbol CP1
- added D3: TVS Diode, symbol ZENER
- added D4: 1N5402, symbol DIODE
- added D5: 1N5821, symbol DIODESCH
- added D6: 1N5820, symbol DIODESCH
- added L1: 20uH, symbol INDUCTOR
- added L2: 150uH, symbol INDUCTOR
- added R3: 5.3k, symbol R
- added R4: 10k, symbol R
- added U2: LM2576, symbol LM257X
- C1: renamed from C201; value 2200uF -> 470uF
- C2: renamed from C202; value 100uF -> 3300uF
- U1: renamed from U201; value LP2950 -> LP2950-30
- renumbered BT201 to BT1, C203 to C3, C204 to C9, D201 to D1, D202 to D2, F201 to F1, R201 to R1, R202 to R2, RSHUNT201 to RSHUNT1, SW201 to SW1, U202 to U3
Connections:
- net labels added: VCC, VDD, VREF
- net labels removed: +3.3V
- wire segments 20 -> 36
Other:
- moved on the sheet: BT1, C1, C2, C3, C9, D1, D2, R1, R2, RSHUNT1, U1, U3

Commit message: first REAL shot at PCB
Parts:
- removed F1: FUSE, symbol FUSE
- removed SW1: SW_POWER, symbol SPST
- C1, C7: footprint (none) -> C2V8
- C2, C4, C6: footprint (none) -> C2V10
- C3, C5, C8, C9: footprint (none) -> C2
- L1: footprint (none) -> INDUCTORV
- R3, R4: footprint (none) -> R4
- RSHUNT1: footprint (none) -> R7
- U1: footprint (none) -> TO-92
- U2: footprint (none) -> TO220
Connections:
- net labels added: +12V
- net labels removed: VCC
- wire segments 36 -> 56
Other:
- note added: "Switch+Fuse OR breakerswitch implied\nhere between BATT+ and connector terminal\n"
- moved on the sheet: C1, C2, C3, D1, U1

Commit message: second try at PCB layout.  this one might actually work!
Changed lines of the file:
@@
-EESchema Schematic File Version 2  date Fri 08 Jun 2012 10:29:21 PM MDT
+EESchema Schematic File Version 2  date Sun 10 Jun 2012 01:48:40 AM MDT
 LIBS:bryan_custom
 LIBS:rfm12
@@
 Sheet 3 6
 Title ""
-Date "8 jun 2012"
+Date "10 jun 2012"
 Rev ""
 Comp ""
@@
 	5250 4950 5250 4400
 Wire Wire Line
-	8600 4350 7800 4350
-Wire Wire Line
-	7800 4350 7600 4350
+	8600 4350 7600 4350
 Connection ~ 2650 3850
 Connection ~ 6300 3750
 Wire Wire Line
-	9350 3350 9050 3350
-Wire Wire Line
-	9050 3350 7850 3350
+	9350 3350 7850 3350
 Connection ~ 2650 4250
 Wire Wire Line
-	3350 4250 2650 4250
-Wire Wire Line
-	2650 4250 1750 4250
+	3350 4250 1750 4250
 Wire Wire Line
 	1900 3850 1750 3850
@@
 Connection ~ 5500 4400
 Wire Wire Line
-	4800 3850 4550 3850
-Wire Wire Line
-	4550 3850 4150 3850
+	4800 3850 4150 3850
 Wire Wire Line
 	7550 1600 7650 1600
@@
 	7650 1600 7650 1900
 Wire Wire Line
-	7200 4600 7200 4350
-Wire Wire Line
-	7200 4350 7200 3750
-Wire Wire Line
-	7200 3750 7200 2950
-Wire Wire Line
-	7200 2950 7200 1900
+	7200 4600 7200 1900
 Wire Wire Line
 	7800 4150 7800 4350
@@
 	7450 6250 7600 6250
 Wire Wire Line
-	6350 5500 6600 5500
-Wire Wire Line
-	6600 5500 6950 5500
+	6350 5500 6950 5500
 Wire Wire Line
 	5500 4400 5500 4600
@@
 	3350 2950 3700 2950
 Wire Wire Line
-	3550 3850 3350 3850
-Wire Wire Line
-	3350 3850 2650 3850
-Wire Wire Line
-	2650 3850 2500 3850
+	3550 3850 2500 3850
 Connection ~ 3350 3850
 Wire Wire Line
-	6000 3750 6300 3750
+	6000 3750 6800 3750
 Wire Wire Line
-	6300 3750 6600 3750
-Wire Wire Line
-	6600 3750 6800 3750
-Wire Wire Line
-	4550 4400 5250 4400
-Wire Wire Line
-	5250 4400 5300 4400
-Wire Wire Line
-	5300 4400 5500 4400
-Wire Wire Line
-	5500 4400 6000 4400
-Wire Wire Line
-	6000 4400 6600 4400
+	4550 4400 6600 4400
 Connection ~ 6000 4400
 Connection ~ 6600 5500
@@
 	7600 2950 7850 2950
 Wire Wire Line
-	9450 3750 8600 3750
-Wire Wire Line
-	8600 3750 7800 3750
+	9450 3750 7800 3750
 Connection ~ 8600 3750
 $Comp

Commit message: further refined PCB, it has safety switch and fire switch and lots of errors fixed!
Parts:
- added Q3: MOSFET_N, symbol MOSFET_N
Connections:
- net GND: now also Q3.S
- new net GNDPWR: Q3.D
- new net HV_control: Q3.G
Changed lines of the file:
@@
-EESchema Schematic File Version 2  date Sun 10 Jun 2012 01:48:40 AM MDT
+EESchema Schematic File Version 2  date Sun 10 Jun 2012 11:49:54 PM MDT
 LIBS:bryan_custom
 LIBS:rfm12
@@
 Sheet 3 6
 Title ""
-Date "10 jun 2012"
+Date "11 jun 2012"
 Rev ""
 Comp ""
@@
 Comment4 ""
 $EndDescr
+Connection ~ 4400 5600
+$Comp
+L PWR_FLAG #FLG018
+U 1 1 4FD56509
+P 4400 5600
+F 0 "#FLG018" H 4400 5870 30  0001 C CNN
+F 1 "PWR_FLAG" H 4400 5830 30  0000 C CNN
+	1    4400 5600
+	0    1    1    0
+$EndComp
+Wire Wire Line
+	4400 5750 4400 5350
+Wire Wire Line
+	4400 6150 4400 6300
 Wire Wire Line
 	8450 3500 8450 3400
@@
 Connection ~ 7850 2950
 Connection ~ 7300 4900
-Connection ~ 4750 4950
 Connection ~ 7300 4900
 Connection ~ 7200 4600
 Connection ~ 5250 4400
 Wire Wire Line
-	4750 4950 5250 4950
-Wire Wire Line
-	5250 4950 5250 4400
+	5250 4400 5250 5050
 Wire Wire Line
 	8600 4350 7600 4350
@@
 Connection ~ 6300 3750
 Wire Wire Line
-	9350 3350 7850 3350
+	7850 3350 9350 3350
 Connection ~ 2650 4250
 Wire Wire Line
-	3350 4250 1750 4250
+	1750 4250 3350 4250
 Wire Wire Line
 	1900 3850 1750 3850
@@
 	6000 4000 6000 3750
 Wire Wire Line
-	3350 3750 3350 3850
+	3350 3850 3350 3750
 Wire Wire Line
 	3350 3350 4700 3350
@@
 Connection ~ 5500 4400
 Wire Wire Line
-	4800 3850 4150 3850
+	4150 3850 4800 3850
 Wire Wire Line
 	7550 1600 7650 1600
@@
 	7450 6250 7600 6250
 Wire Wire Line
-	6350 5500 6950 5500
+	6950 5500 6350 5500
 Wire Wire Line
 	5500 4400 5500 4600
@@
 	3350 2950 3700 2950
 Wire Wire Line
-	3550 3850 2500 3850
+	2500 3850 3550 3850
 Connection ~ 3350 3850
 Wire Wire Line
 	6000 3750 6800 3750
 Wire Wire Line
-	4550 4400 6600 4400
+	6600 4400 4550 4400
 Connection ~ 6000 4400
 Connection ~ 6600 5500
@@
 	7600 2950 7850 2950
 Wire Wire Line
-	9450 3750 7800 3750
+	7800 3750 9450 3750
 Connection ~ 8600 3750
-$Comp
-L PWR_FLAG #FLG018
+Wire Wire Line
+	6850 4350 7200 4350
+Wire Wire Line
+	4100 5950 3950 5950
+$Comp
+L GNDPWR #PWR019
+U 1 1 4FD55EA4
+P 4400 5350
+F 0 "#PWR019" H 4400 5400 40  0001 C CNN
+F 1 "GNDPWR" H 4400 5270 40  0000 C CNN
+	1    4400 5350
+	-1   0    0    1
+$EndComp
+Text HLabel 3950 5950 0    60   Input ~ 0
+HV_control
+$Comp
+L GND #PWR020
+U 1 1 4FD55DB8
+P 4400 6300
+F 0 "#PWR020" H 4400 6300 30  0001 C CNN
+F 1 "GND" H 4400 6230 30  0001 C CNN
+	1    4400 6300
+	1    0    0    -1
+$EndComp
+$Comp
+L +12V #PWR021
+U 1 1 4FD17D59
+P 6850 4350
+F 0 "#PWR021" H 6850 4300 20  0001 C CNN
+F 1 "+12V" H 6850 4450 30  0000 C CNN
+	1    6850 4350
+	1    0    0    -1
+$EndComp
+$Comp
+L MOSFET_N Q3
+U 1 1 4FD5598B
+P 4300 5950
+F 0 "Q3" H 4310 6120 60  0000 R CNN
+F 1 "MOSFET_N" H 4310 5800 60  0000 R CNN
+	1    4300 5950
+	1    0    0    -1
+$EndComp
+$Comp
+L PWR_FLAG #FLG022
 U 1 1 4FD18A2D
 P 1450 3600
-F 0 "#FLG018" H 1450 3870 30  0001 C CNN
+F 0 "#FLG022" H 1450 3870 30  0001 C CNN
 F 1 "PWR_FLAG" H 1450 3830 30  0000 C CNN
 	1    1450 3600
@@
 $EndComp
 $Comp
-L PWR_FLAG #FLG019
+L PWR_FLAG #FLG023
 U 1 1 4FD1862E
 P 7600 3300
-F 0 "#FLG019" H 7600 3570 30  0001 C CNN
+F 0 "#FLG023" H 7600 3570 30  0001 C CNN
 F 1 "PWR_FLAG" H 7600 3530 30  0000 C CNN
 	1    7600 3300
@@
 $EndComp
 $Comp
-L PWR_FLAG #FLG020
+L PWR_FLAG #FLG024
 U 1 1 4FD1853D
 P 7200 4600
-F 0 "#FLG020" H 7200 4870 30  0001 C CNN
+F 0 "#FLG024" H 7200 4870 30  0001 C CNN
 F 1 "PWR_FLAG" H 7200 4830 30  0000 C CNN
 	1    7200 4600
@@
 $EndComp
 $Comp
-L GND #PWR021
+L GND #PWR025
 U 1 1 4FD18256
-P 4750 4950
-F 0 "#PWR021" H 4750 4950 30  0001 C CNN
-F 1 "GND" H 4750 4880 30  0001 C CNN
-	1    4750 4950
-	1    0    0    -1
-$EndComp
-$Comp
-L +12V #PWR022
-U 1 1 4FD17D59
-P 7200 4350
-F 0 "#PWR022" H 7200 4300 20  0001 C CNN
-F 1 "+12V" H 7200 4450 30  0000 C CNN
-	1    7200 4350
-	0    -1   -1   0
-$EndComp
-$Comp
-L VDD #PWR023
+P 5250 5050
+F 0 "#PWR025" H 5250 5050 30  0001 C CNN
+F 1 "GND" H 5250 4980 30  0001 C CNN
+	1    5250 5050
+	1    0    0    -1
+$EndComp
+$Comp
+L VDD #PWR026
 U 1 1 4FCD406E
 P 1750 3600
-F 0 "#PWR023" H 1750 3700 30  0001 C CNN
+F 0 "#PWR026" H 1750 3700 30  0001 C CNN
 F 1 "VDD" H 1750 3710 30  0000 C CNN
 	1    1750 3600
@@
 $EndComp
 $Comp
-L GND #PWR024
+L GND #PWR027
 U 1 1 4F87A33D
 P 6300 3350
-F 0 "#PWR024" H 6300 3350 30  0001 C CNN
+F 0 "#PWR027" H 6300 3350 30  0001 C CNN
 F 1 "GND" H 6300 3280 30  0001 C CNN
 	1    6300 3350
@@
 $EndComp
 $Comp
-L VDD #PWR025
+L VDD #PWR028
 U 1 1 4F879E14
 P 6600 5500
-F 0 "#PWR025" H 6600 5600 30  0001 C CNN
+F 0 "#PWR028" H 6600 5600 30  0001 C CNN
 F 1 "VDD" H 6600 5610 30  0000 C CNN
 	1    6600 5500
@@
 $EndComp
 $Comp
-L GND #PWR026
+L GND #PWR029
 U 1 1 4F879CC0
 P 3350 4250
-F 0 "#PWR026" H 3350 4250 30  0001 C CNN
+F 0 "#PWR029" H 3350 4250 30  0001 C CNN
 F 1 "GND" H 3350 4180 30  0001 C CNN
 	1    3350 4250
@@
 $EndComp
 $Comp
-L GND #PWR027
+L GND #PWR030
 U 1 1 4F879849
 P 3700 2950
-F 0 "#PWR027" H 3700 2950 30  0001 C CNN
+F 0 "#PWR030" H 3700 2950 30  0001 C CNN
 F 1 "GND" H 3700 2880 30  0001 C CNN
 	1    3700 2950
@@
 $EndComp
 $Comp
-L GND #PWR028
+L GND #PWR031
 U 1 1 4F86764B
 P 5500 4600
-F 0 "#PWR028" H 5500 4600 30  0001 C CNN
+F 0 "#PWR031" H 5500 4600 30  0001 C CNN
 F 1 "GND" H 5500 4530 30  0001 C CNN
 	1    5500 4600
@@
 NOTE: Enhanced Voltage reference is \noptional.  If not used, connect AVR \nAREF and TSC888 VIN to the digital\nsupply (3.3 to 3.6V)
 $Comp
-L GND #PWR029
+L GND #PWR032
 U 1 1 4F25D8AC
 P 9450 3750
-F 0 "#PWR029" H 9450 3750 30  0001 C CNN
+F 0 "#PWR032" H 9450 3750 30  0001 C CNN
 F 1 "GND" H 9450 3680 30  0001 C CNN
 	1    9450 3750
@@
 $EndComp
 $Comp
-L GND #PWR030
+L GND #PWR033
 U 1 1 4E87E2F9
 P 7850 2550
-F 0 "#PWR030" H 7850 2550 30  0001 C CNN
+F 0 "#PWR033" H 7850 2550 30  0001 C CNN
 F 1 "GND" H 7850 2480 30  0001 C CNN
 	1    7850 2550
@@
 $EndComp
 $Comp
-L GND #PWR031
+L GND #PWR034
 U 1 1 4F25D8A7
 P 6350 5900
-F 0 "#PWR031" H 6350 5900 30  0001 C CNN
+F 0 "#PWR034" H 6350 5900 30  0001 C CNN
 F 1 "GND" H 6350 5830 30  0001 C CNN
 	1    6350 5900
@@
 $EndComp
 $Comp
-L GND #PWR032
+L GND #PWR035
 U 1 1 4E55D85B
 P 8000 5400
-F 0 "#PWR032" H 8000 5400 30  0001 C CNN
+F 0 "#PWR035" H 8000 5400 30  0001 C CNN
 F 1 "GND" H 8000 5330 30  0001 C CNN
 	1    8000 5400
@@
 $EndComp
 $Comp
-L GND #PWR033
+L GND #PWR036
 U 1 1 4EAB7ADD
 P 8450 3500
-F 0 "#PWR033" H 8450 3500 30  0001 C CNN
+F 0 "#PWR036" H 8450 3500 30  0001 C CNN
 F 1 "GND" H 8450 3430 30  0001 C CNN
 	1    8450 3500
@@
 $EndComp
 $Comp
-L GND #PWR034
+L GND #PWR037
 U 1 1 4F25D8A0
 P 8050 1900
-F 0 "#PWR034" H 8050 1900 30  0001 C CNN
+F 0 "#PWR037" H 8050 1900 30  0001 C CNN
 F 1 "GND" H 8050 1830 30  0001 C CNN
 	1    8050 1900
