File: CRASH-launcher/docs/kicad-bryan_4chan/power.sch (KiCad schematic (older format))
At the start: 27 parts, among them Q3 MOSFET_N, U1 LP2950-30, U2 LM2576, U3 TSC888

Commit message: lots of revs, breakout board
Parts:
- added D11, D12, D13: LED, symbol LED
- added R15, R16, R17: 1k, symbol R
- added R18: 1.8k, symbol R
- added TST-VDD1: TST-VDD, symbol TST
- added TST-VREF1: TST-VREF, symbol TST
- C2, C4: value 3300uF -> 100uF
Connections:
- net +12V: now also R18.1
- net GND: now also R15.1, R16.1, R17.1
- net GNDPWR: now also D12.2 (K)
- net HV_control: now also R15.2
- net VDD: now also D11.1 (A), TST-VDD1.1
- net VREF: now also D13.1 (A), TST-VREF1.1
- new net: D11.2 (K), R17.2
- new net: D12.1 (A), R18.2
- new net: D13.2 (K), R16.2
