File: hardware-designs/candleFX/candleFX.kicad_pcb (KiCad board)
At the start: 2 copper layers, 63.5 x 54.6 mm, 16 parts, among them IC1 ATTINY85-P, U1 OPTO-TRIAC, U2 TRIAC, U3 LP2950

Commit message: today!
Parts:
- removed RV3: 20k, Potentiometer_RevB_02Aug2010:Potentiometer_Trimmer-Piher_PT15-V15_horizontal_RevA_02Aug2010
- added D3: 1n4148, discret:D3, F.Cu at (183.1, 96.5)
- added R3: 1k, discret:R3-LARGE_PADS, F.Cu at (174.0, 86.6)
- added R4: 10k, discret:R3-LARGE_PADS, F.Cu at (177.0, 93.0)
