File: hardware-designs/candleFX/candleFX.sch (KiCad schematic (older format))
At the start: 16 parts, among them IC1 ATTINY85-P, U1 OPTO-TRIAC, U2 TRIAC, U3 LP2950

Commit message: today!
Parts:
- removed RV3: 20k, symbol POT
- added D3: 1n4148, symbol DIODE
- added R3: 1k, symbol R
- added R4: 10k, symbol R
Connections:
- net GND: now also D3.2 (K), R3.2
- net at IC1.7 (PB2(SCK/USCK/SCL/T0/INT0/ADC1/PCINT2)): now also D3.1 (A), R3.1, R4.2
- net at D1.3 (+), D2.1 (A): now also R4.1
Other:
- moved on the sheet: L1, R1, R2, U1, U2
Changed lines of the file:
@@
 L OPTO-TRIAC U1
 U 1 1 5350C1A2
-P 4500 3550
-F 0 "U1" H 4700 3850 60  0000 C CNN
-F 1 "OPTO-TRIAC" H 4600 3250 60  0000 C CNN
-F 2 "" H 4500 3550 60  0000 C CNN
-F 3 "" H 4500 3550 60  0000 C CNN
-	1    4500 3550
+P 5800 3550
+F 0 "U1" H 6000 3850 60  0000 C CNN
+F 1 "OPTO-TRIAC" H 5900 3250 60  0000 C CNN
+F 2 "" H 5800 3550 60  0000 C CNN
+F 3 "" H 5800 3550 60  0000 C CNN
+	1    5800 3550
 	1    0    0    -1
 $EndComp
@@
 U 1 1 5350C1D5
 P 3300 2750
-F 0 "IC1" H 2150 3150 40  0000 C CNN
+F 0 "IC1" H 1050 3250 40  0000 C CNN
 F 1 "ATTINY85-P" H 4300 2350 40  0000 C CNN
 F 2 "DIP8" H 4300 2750 35  0000 C CIN
@@
 L TRIAC U2
 U 1 1 5350C1F3
-P 6200 3550
-F 0 "U2" H 5950 3900 70  0000 C CNN
-F 1 "TRIAC" H 5900 3300 60  0000 C CNN
-F 2 "" H 6200 3550 60  0000 C CNN
-F 3 "" H 6200 3550 60  0000 C CNN
-	1    6200 3550
+P 7500 3550
+F 0 "U2" H 7250 3900 70  0000 C CNN
+F 1 "TRIAC" H 7200 3300 60  0000 C CNN
+F 2 "" H 7500 3550 60  0000 C CNN
+F 3 "" H 7500 3550 60  0000 C CNN
+	1    7500 3550
 	1    0    0    -1
 $EndComp
@@
 L R R1
 U 1 1 5350C20D
-P 5950 2950
-F 0 "R1" H 5950 2850 40  0000 C CNN
-F 1 "100" H 5950 3000 40  0000 C CNN
-F 2 "" V 5880 2950 30  0000 C CNN
-F 3 "" H 5950 2950 30  0000 C CNN
-	1    5950 2950
+P 7250 2950
+F 0 "R1" H 7250 2850 40  0000 C CNN
+F 1 "100" H 7250 3000 40  0000 C CNN
+F 2 "" V 7180 2950 30  0000 C CNN
+F 3 "" H 7250 2950 30  0000 C CNN
+	1    7250 2950
 	-1   0    0    1
 $EndComp
@@
 L INDUCTOR L1
 U 1 1 5350C32F
-P 7200 3250
-F 0 "L1" V 7150 3250 40  0000 C CNN
-F 1 "LAMP" V 7300 3250 40  0000 C CNN
-F 2 "" H 7200 3250 60  0000 C CNN
-F 3 "" H 7200 3250 60  0000 C CNN
-	1    7200 3250
+P 8500 3250
+F 0 "L1" V 8450 3250 40  0000 C CNN
+F 1 "LAMP" V 8600 3250 40  0000 C CNN
+F 2 "" H 8500 3250 60  0000 C CNN
+F 3 "" H 8500 3250 60  0000 C CNN
+	1    8500 3250
 	1    0    0    -1
 $EndComp
@@
 $EndComp
 $Comp
-L GND #PWR01
+L GND #PWR2
 U 1 1 5358882C
 P 650 2250
-F 0 "#PWR01" H 650 2250 30  0001 C CNN
+F 0 "#PWR2" H 650 2250 30  0001 C CNN
 F 1 "GND" H 650 2180 30  0001 C CNN
 F 2 "" H 650 2250 60  0000 C CNN
@@
 L R R2
 U 1 1 53588C7B
-P 3400 3650
-F 0 "R2" H 3440 3720 50  0000 C CNN
-F 1 "330" H 3430 3580 50  0000 C CNN
-F 2 "" H 3400 3650 60  0000 C CNN
-F 3 "" H 3400 3650 60  0000 C CNN
-	1    3400 3650
-	1    0    0    -1
-$EndComp
-$Comp
-L GND #USGND02
+P 5000 3850
+F 0 "R2" H 5040 3920 50  0000 C CNN
+F 1 "330" H 5030 3780 50  0000 C CNN
+F 2 "" H 5000 3850 60  0000 C CNN
+F 3 "" H 5000 3850 60  0000 C CNN
+	1    5000 3850
+	0    -1   -1   0
+$EndComp
+$Comp
+L GND #USGND6
 U 1 1 53588CA5
-P 3200 3850
-F 0 "#USGND02" H 2900 3550 60  0001 C CNN
-F 1 "GND" H 3200 3715 60  0000 C CNN
-F 2 "" H 3200 3850 60  0000 C CNN
-F 3 "" H 3200 3850 60  0000 C CNN
-	1    3200 3850
+P 5000 4250
+F 0 "#USGND6" H 4700 3950 60  0001 C CNN
+F 1 "GND" H 5000 4115 60  0000 C CNN
+F 2 "" H 5000 4250 60  0000 C CNN
+F 3 "" H 5000 4250 60  0000 C CNN
+	1    5000 4250
 	1    0    0    -1
 $EndComp
@@
 $EndComp
 $Comp
-L POT RV3
-U 1 1 53588D33
-P 5600 2050
-F 0 "RV3" H 5600 1950 50  0000 C CNN
-F 1 "20k" H 5600 2050 50  0000 C CNN
-F 2 "" H 5600 2050 60  0000 C CNN
-F 3 "" H 5600 2050 60  0000 C CNN
-	1    5600 2050
-	-1   0    0    1
-$EndComp
-$Comp
-L GND #USGND03
-U 1 1 53588D88
-P 5350 2100
-F 0 "#USGND03" H 5050 1800 60  0001 C CNN
-F 1 "GND" H 5350 1965 60  0000 C CNN
-F 2 "" H 5350 2100 60  0000 C CNN
-F 3 "" H 5350 2100 60  0000 C CNN
-	1    5350 2100
-	1    0    0    -1
-$EndComp
-$Comp
-L GND #USGND04
+L GND #USGND2
 U 1 1 53588DC2
 P 4300 2050
-F 0 "#USGND04" H 4000 1750 60  0001 C CNN
+F 0 "#USGND2" H 4000 1750 60  0001 C CNN
 F 1 "GND" H 4300 1915 60  0000 C CNN
 F 2 "" H 4300 2050 60  0000 C CNN
@@
 $EndComp
 $Comp
-L GND #USGND05
+L GND #USGND1
 U 1 1 53588DEC
 P 3650 1850
-F 0 "#USGND05" H 3350 1550 60  0001 C CNN
+F 0 "#USGND1" H 3350 1550 60  0001 C CNN
 F 1 "GND" H 3650 1715 60  0000 C CNN
 F 2 "" H 3650 1850 60  0000 C CNN
@@
 $EndComp
 $Comp
-L GND #USGND06
+L GND #USGND8
 U 1 1 53588FB5
 P 3750 6550
-F 0 "#USGND06" H 3450 6250 60  0001 C CNN
+F 0 "#USGND8" H 3450 6250 60  0001 C CNN
 F 1 "GND" H 3750 6415 60  0000 C CNN
 F 2 "" H 3750 6550 60  0000 C CNN
@@
 Wire Wire Line
 	3750 6550 3750 6350
-Connection ~ 6200 2950
-Wire Wire Line
-	5600 2200 5600 2450
-Wire Wire Line
-	5350 2050 5350 2100
-Wire Wire Line
-	5100 3750 5700 3750
-Wire Wire Line
-	6150 2950 7200 2950
-Wire Wire Line
-	5100 3350 5100 2950
-Wire Wire Line
-	5100 2950 5750 2950
-Wire Wire Line
-	7200 5500 7200 3550
+Connection ~ 7500 2950
+Wire Wire Line
+	6400 3750 7000 3750
+Wire Wire Line
+	7450 2950 8500 2950
+Wire Wire Line
+	6400 3350 6400 2950
+Wire Wire Line
+	6400 2950 7050 2950
+Wire Wire Line
+	8500 5500 8500 3550
 Wire Wire Line
 	2400 5500 2900 5500
 Wire Wire Line
-	4600 5500 7200 5500
+	4600 5500 8500 5500
 Connection ~ 4700 5500
 Wire Wire Line
 	2900 5500 2900 6950
 Wire Wire Line
-	2900 6950 6200 6950
-Wire Wire Line
-	6200 6950 6200 3800
-Wire Wire Line
-	6200 2950 6200 3150
+	2900 6950 7500 6950
+Wire Wire Line
+	7500 6950 7500 3800
+Wire Wire Line
+	7500 2950 7500 3150
 Wire Wire Line
 	1750 4650 3000 4650
@@
 	800  3450 800  2650
 Wire Wire Line
-	3600 3650 3850 3650
-Wire Wire Line
-	3200 3650 3200 3850
-Wire Wire Line
-	3850 3350 3850 2650
-Wire Wire Line
-	3850 2650 3500 2650
-Wire Wire Line
-	4150 1800 5850 1800
+	5000 3650 5150 3650
+Wire Wire Line
+	5150 2650 5150 3350
+Wire Wire Line
+	3500 2650 5150 2650
 Wire Wire Line
 	4800 1800 4800 2000
 Wire Wire Line
-	5850 1800 5850 2050
-Connection ~ 4800 1800
-Wire Wire Line
 	4300 2000 4300 2050
 Wire Wire Line
@@
 Wire Wire Line
 	4550 2350 3500 2350
-Wire Wire Line
-	5600 2450 3500 2450
 NoConn ~ 3500 2550
 NoConn ~ 3500 2150
@@
 	650  2150 650  2250
 $Comp
-L GND #USGND07
+L GND #USGND4
 U 1 1 53604EB7
 P 2200 4250
-F 0 "#USGND07" H 1900 3950 60  0001 C CNN
+F 0 "#USGND4" H 1900 3950 60  0001 C CNN
 F 1 "GND" H 2200 4115 60  0000 C CNN
 F 2 "" H 2200 4250 60  0000 C CNN
@@
 Connection ~ 2500 4650
 $Comp
-L PWR_FLAG #FLG08
+L PWR_FLAG #FLG1
 U 1 1 53605C9A
 P 2350 4650
-F 0 "#FLG08" H 2350 4745 30  0001 C CNN
+F 0 "#FLG1" H 2350 4745 30  0001 C CNN
 F 1 "PWR_FLAG" H 2350 4830 30  0000 C CNN
 F 2 "" H 2350 4650 60  0000 C CNN
@@
 Connection ~ 2350 4650
 $Comp
-L +12V #PWR09
+L +12V #PWR5
 U 1 1 536057C3
 P 4700 5350
-F 0 "#PWR09" H 4700 5300 20  0001 C CNN
+F 0 "#PWR5" H 4700 5300 20  0001 C CNN
 F 1 "+12V" H 4700 5450 30  0000 C CNN
 F 2 "" H 4700 5350 60  0000 C CNN
@@
 	4700 5500 4700 5350
 $Comp
-L PWR_FLAG #FLG010
+L PWR_FLAG #FLG2
 U 1 1 5360580B
 P 4900 5400
-F 0 "#FLG010" H 4900 5495 30  0001 C CNN
+F 0 "#FLG2" H 4900 5495 30  0001 C CNN
 F 1 "PWR_FLAG" H 4900 5580 30  0000 C CNN
 F 2 "" H 4900 5400 60  0000 C CNN
@@
 Connection ~ 4900 5500
 $Comp
-L -12V #PWR011
+L -12V #PWR6
 U 1 1 5360584B
 P 2400 5500
-F 0 "#PWR011" H 2400 5630 20  0001 C CNN
+F 0 "#PWR6" H 2400 5630 20  0001 C CNN
 F 1 "-12V" H 2400 5600 30  0000 C CNN
 F 2 "" H 2400 5500 60  0000 C CNN
@@
 $EndComp
 $Comp
-L PWR_FLAG #FLG012
+L PWR_FLAG #FLG3
 U 1 1 536058F1
 P 2700 5500
-F 0 "#FLG012" H 2700 5595 30  0001 C CNN
+F 0 "#FLG3" H 2700 5595 30  0001 C CNN
 F 1 "PWR_FLAG" H 2700 5680 30  0000 C CNN
 F 2 "" H 2700 5500 60  0000 C CNN
@@
 Connection ~ 2700 5500
 $Comp
-L +9V #PWR013
+L +9V #PWR4
 U 1 1 53605911
 P 2500 4550
-F 0 "#PWR013" H 2500 4520 20  0001 C CNN
+F 0 "#PWR4" H 2500 4520 20  0001 C CNN
 F 1 "+9V" H 2500 4660 30  0000 C CNN
 F 2 "" H 2500 4550 60  0000 C CNN
@@
 VCC
 $Comp
-L VCC #PWR014
+L VCC #PWR3
 U 1 1 536060DB
 P 1300 3450
-F 0 "#PWR014" H 1300 3550 30  0001 C CNN
+F 0 "#PWR3" H 1300 3550 30  0001 C CNN
 F 1 "VCC" H 1300 3550 30  0000 C CNN
 F 2 "" H 1300 3450 60  0000 C CNN
@@
 Connection ~ 1300 3450
 $Comp
-L VCC #PWR015
+L VCC #PWR1
 U 1 1 536060F1
 P 4800 1800
-F 0 "#PWR015" H 4800 1900 30  0001 C CNN
+F 0 "#PWR1" H 4800 1900 30  0001 C CNN
 F 1 "VCC" H 4800 1900 30  0000 C CNN
 F 2 "" H 4800 1800 60  0000 C CNN
@@
 Connection ~ 2200 3150
 $Comp
-L GND #USGND016
+L GND #USGND3
 U 1 1 5360630E
 P 2500 3450
-F 0 "#USGND016" H 2200 3150 60  0001 C CNN
+F 0 "#USGND3" H 2200 3150 60  0001 C CNN
 F 1 "GND" H 2500 3315 60  0000 C CNN
 F 2 "" H 2500 3450 60  0000 C CNN
@@
 $EndComp
 Wire Wire Line
-	3400 4650 3750 4650
+	3400 4650 4150 4650
 $Comp
 L C C4
@@
 $EndComp
 Wire Wire Line
-	2800 4650 2800 4250
+	2800 4250 2800 4650
 Connection ~ 2800 4500
 Wire Wire Line
 	3200 4250 3200 4500
 $Comp
-L GND #USGND017
+L GND #USGND7
 U 1 1 53606423
 P 3650 4400
-F 0 "#USGND017" H 3350 4100 60  0001 C CNN
+F 0 "#USGND7" H 3350 4100 60  0001 C CNN
 F 1 "GND" H 3650 4265 60  0000 C CNN
 F 2 "" H 3650 4400 60  0000 C CNN
@@
 	3650 4250 3650 4400
 Connection ~ 2800 4650
+Wire Wire Line
+	5000 4050 5000 4250
+Wire Wire Line
+	4150 4650 4150 4200
+$Comp
+L R R4
+U 1 1 54347BF2
+P 4150 4000
+F 0 "R4" H 4190 4070 50  0000 C CNN
+F 1 "10k" H 4180 3930 50  0000 C CNN
+F 2 "" H 4150 4000 60  0000 C CNN
+F 3 "" H 4150 4000 60  0000 C CNN
+	1    4150 4000
+	0    -1   -1   0
+$EndComp
+$Comp
+L R R3
+U 1 1 54347C06
+P 4350 3700
+F 0 "R3" H 4390 3770 50  0000 C CNN
+F 1 "1k" H 4380 3630 50  0000 C CNN
+F 2 "" H 4350 3700 60  0000 C CNN
+F 3 "" H 4350 3700 60  0000 C CNN
+	1    4350 3700
+	1    0    0    -1
+$EndComp
+$Comp
+L DIODE D3
+U 1 1 54347C1A
+P 4350 3400
+F 0 "D3" H 4350 3500 40  0000 C CNN
+F 1 "1n4148" H 4350 3300 40  0000 C CNN
+F 2 "" H 4350 3400 60  0000 C CNN
+F 3 "" H 4350 3400 60  0000 C CNN
+	1    4350 3400
+	1    0    0    -1
+$EndComp
+Wire Wire Line
+	4150 2450 4150 3800
+Connection ~ 4150 3700
+Wire Wire Line
+	4550 3400 4550 4250
+Connection ~ 4550 3700
+Connection ~ 4150 3400
+Wire Wire Line
+	4800 1800 4150 1800
+Connection ~ 4800 1800
+Wire Wire Line
+	3500 2450 4150 2450
+$Comp
+L GND #USGND5
+U 1 1 54347E28
+P 4550 4250
+F 0 "#USGND5" H 4250 3950 60  0001 C CNN
+F 1 "GND" H 4550 4115 60  0000 C CNN
+F 2 "" H 4550 4250 60  0000 C CNN
+F 3 "" H 4550 4250 60  0000 C CNN
+	1    4550 4250
+	1    0    0    -1
+$EndComp
 $EndSCHEMATC
